File: Fox_Rover/_autosave-FoxRobot.kicad_pcb (KiCad board)
At the start: 2 copper layers, 38 parts, among them J1 Screw_Terminal_01x02, J2 XT60-M_Green, J3 XT60-M_Red, J4 Screw_Terminal_01x02, J5 Conn_02x10_Odd_Even, J6 Screw_Terminal_01x02, J7 Conn_02x10_Odd_Even, K1 40.52.7.012.0000, K2 G2RK-1_12DC, K3 ADJH23005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

Commit message: PCB design suitable
Parts:
- removed REF** (x4): MountingHole_3.2mm_M3_DIN965_Pad, MountingHole:MountingHole_3.2mm_M3_DIN965_Pad
- added H1: MountingHole, MountingHole:MountingHole_3.2mm_M3_ISO7380_Pad_TopBottom, F.Cu at (19.1, 24.1)
- added H2: MountingHole, MountingHole:MountingHole_3.2mm_M3_ISO7380_Pad_TopBottom, F.Cu at (100.9, 28.2)
- added H3: MountingHole, MountingHole:MountingHole_3.2mm_M3_ISO7380_Pad_TopBottom, F.Cu at (33.0, 119.4)
- added H4: MountingHole, MountingHole:MountingHole_3.2mm_M3_ISO7380_Pad_TopBottom, F.Cu at (109.2, 119.4)
- moved J7 7.62 mm to (88.9, 15.2)
- moved J5 7.24 mm to (19.7, 15.2)
- moved J4 5.33 mm to (76.7, 19.1)
- moved J1 4.83 mm to (64.0, 19.1)
- moved J6 4.83 mm to (50.8, 19.1)
Routing:
- net Net-(J3-Pad2): track 216.3 -> 121.6 mm
- net GND: track 235.9 -> 298.0 mm
- net Net-(K3-Pad1): track 101.0 -> 63.1 mm, vias 0 -> 1
- net Net-(J6-Pad2): track 148.4 -> 113.2 mm
- net Net-(Q9-Pad2): track 29.7 -> 64.4 mm, vias 1 -> 0
- net Net-(Q8-Pad2): track 32.1 -> 56.3 mm
- net Net-(J2-Pad2): track 178.3 -> 154.5 mm, vias 0 -> 1
- net Net-(K3-Pad2): track 86.2 -> 64.0 mm, vias 0 -> 1
- net Net-(K2-Pad2): track 67.7 -> 88.2 mm
- net Net-(Q6-Pad2): track 54.9 -> 36.8 mm
- net /A3: track 101.3 -> 111.6 mm
- net Net-(Q4-Pad2): track 35.7 -> 45.2 mm
- net /A4: track 94.4 -> 102.5 mm
- net Net-(K2-Pad1): track 57.0 -> 64.9 mm
- net Net-(J4-Pad2): track 90.4 -> 96.8 mm
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Other:
- board text added: "24V+"
